File: layouts/default/default.kicad_pcb (KiCad board)
At the start: 2 copper layers, 194 parts

Commit message: build(ato): add PCB layout and auto-picked component packages from first successful ato build
Add KiCad PCB layout (default.kicad_pcb), footprint library table,
and two auto-generated component packages:
- Murata BLM15AG601SN1D ferrite bead
- UNI-ROYAL 0402WGF1200TCE 120 ohm CAN termination resistor

Co-Authored-By: Claude Opus 4.6 (1M context) <noreply@anthropic.com>
Parts:
- added C92: 100nF ±10%, Samsung_Electro_Mechanics_CL05B104KO5NNNC:C0402, F.Cu at (37.8, 0.10)
- added C93: 100nF ±10%, Samsung_Electro_Mechanics_CL05B104KO5NNNC:C0402, F.Cu at (47.8, 0.10)
- added C94: 100nF ±10%, Samsung_Electro_Mechanics_CL05B104KO5NNNC:C0402, F.Cu at (60.0, -50.0)
- added C95: 100nF ±10%, Samsung_Electro_Mechanics_CL05B104KO5NNNC:C0402, F.Cu at (60.0, -55.0)
- added C96: 100nF ±10%, Samsung_Electro_Mechanics_CL05B104KO5NNNC:C0402, F.Cu at (60.0, -70.0)
- added C97: 100nF ±10%, Samsung_Electro_Mechanics_CL05B104KO5NNNC:C0402, F.Cu at (60.0, -75.0)
- added C98: 100nF ±10%, Samsung_Electro_Mechanics_CL05B104KO5NNNC:C0402, F.Cu at (60.0, -90.0)
- added C99: 100nF ±10%, Samsung_Electro_Mechanics_CL05B104KO5NNNC:C0402, F.Cu at (60.0, -105.0)
- added R78: 100Ω ±1%, UNI_ROYAL_0402WGF1000TCE:R0402, F.Cu at (60.0, -25.0)
- added R79: 8.06kΩ ±1%, YAGEO_RC0402FR_078K06L:R0402, F.Cu at (60.0, -30.0)
- added R80: 10kΩ ±1%, UNI_ROYAL_0402WGF1002TCE:R0402, F.Cu at (60.0, -35.0)
- added R81: 10kΩ ±1%, UNI_ROYAL_0402WGF1002TCE:R0402, F.Cu at (60.0, -60.0)
- added R82: 10kΩ ±1%, UNI_ROYAL_0402WGF1002TCE:R0402, F.Cu at (60.0, -65.0)
- added R83: 10kΩ ±1%, UNI_ROYAL_0402WGF1002TCE:R0402, F.Cu at (60.0, -80.0)
- added R84: 10kΩ ±1%, UNI_ROYAL_0402WGF1002TCE:R0402, F.Cu at (60.0, -85.0)
- added R85: 10kΩ ±1%, UNI_ROYAL_0402WGF1002TCE:R0402, F.Cu at (60.0, -95.0)
- added R86: 120Ω ±1%, UNI_ROYAL_0402WGF1200TCE:R0402, F.Cu at (60.0, -100.0)
- added R87: 100Ω ±1%, UNI_ROYAL_0402WGF1000TCE:R0402, F.Cu at (60.0, -110.0)
- added U22: , Texas_Instruments_TS5A22362DGSR:VSSOP-10_L3.0-W3.0-P0.50-LS4.9-BL, F.Cu at (40.0, 0.00)
- added U23: , Texas_Instruments_TS5A22362DGSR:VSSOP-10_L3.0-W3.0-P0.50-LS4.9-BL, F.Cu at (50.0, 0.00)
- added U24: , Texas_Instruments_ISO7741DBQR:SSOP-16_L5.3-W3.4-P0.65-LS5.2, F.Cu at (20.0, 0.00)
- added U25: , Texas_Instruments_ISO7741DBQR:SSOP-16_L5.3-W3.4-P0.65-LS5.2, F.Cu at (30.0, 0.00)
- added U26: , Texas_Instruments_SN65HVD230DR:SOIC-8_L4.9-W3.9-P1.27-LS6.0-BL, F.Cu at (0.00, 0.00)
- added U27: , Texas_Instruments_SN74HC138PWR:TSSOP-16_L5.0-W4.4-P0.65-LS6.4-BL, F.Cu at (10.0, 0.00)
- C23: value 270pF ±10% -> 10pF ±5%; footprint STE_R06B1B271KN0B0S0N0:CAP-TH_L6.0-W2.5-P5.00-D1.0 -> CCTC_TCC0402C0G100J500AT:C0402
- C67: value 100nF ±10% -> 1nF ±10%; footprint Samsung_Electro_Mechanics_CL05B104KO5NNNC:C0402 -> YAGEO_CC0402KRX7R9BB102:C0402
- R21, R22, R32: value 100mΩ ±5% -> L {ℝ+}H; footprint UNI_ROYAL_0402WGJ010KTCE:R0402 -> Murata_Electronics_BLM15AG601SN1D:L0402
- R9: value 8.06kΩ ±1% -> 1kΩ ±1%; footprint YAGEO_RC0402FR_078K06L:R0402 -> UNI_ROYAL_0402WGF1001TCE:R0402
- moved R9 147.7 mm to (60.0, -5.00)
- moved C9 145.9 mm to (60.0, 0.00)
- moved C67 92.2 mm to (60.0, -20.0)
- moved C66 91.4 mm to (60.0, -15.0)
- moved C23 10.2 mm to (60.0, -10.0), turned to 0 degrees
Connections:
- net 16 renamed io[46]-16
- net 6 renamed _inductor_2-6
- net 7 renamed filter_switch-enables[1]-7
- net CS renamed gpio[17]-line
- net cell_enable-line renamed gpio[11]-line
- C23 pad 1: power_neg-hv -> comp_c0-power-hv
- C23 pad 2: lv_N -> lv
- C28 pad 1: pi_cap_digital-power-hv -> hv
- C54 pad 1: power_3v3-hv -> wifi_bypass_cap-power-hv
- C57 pad 1: power_3v3-hv -> wifi_bypass_cap-power-hv
- C61 pad 1: power_3v3-hv -> wifi_bypass_cap-power-hv
- C65 pad 1: pi_cap_digital-power-hv -> hv
- C66 pad 1: power_5v-hv -> comp_c1-power-hv
- C66 pad 2: power_neg-hv -> lv
- C67 pad 1: pi_cap_digital-power-hv -> comp_c2-power-hv
- C67 pad 2: lv_N -> lv
- C71 pad 1: pi_cap_digital-power-hv -> hv
- C9 pad 1: comp_capacitor-power-hv -> hv
- C9 pad 2: lv -> lv_N
- R21 pad 2: pi_cap_digital-power-hv -> hv
- R32 pad 1: power_3v3-hv -> wifi_bypass_cap-power-hv
- R34 pad 1: pi_cap_digital-power-hv -> hv
- R36 pad 1: pi_cap_digital-power-hv -> hv
- R70 pad 1: power_3v3-hv -> wifi_bypass_cap-power-hv
- R9 pad 1: comp_capacitor-power-hv -> gpio[25]-line
- R9 pad 2: lv -> lv_N
- U1 pad 12: (no net) -> 12
- U1 pad 13: DRDY -> gpio[16]-line
- U10 pad 5: power_3v3-hv -> wifi_bypass_cap-power-hv
- U14 pad 3: comp_capacitor-power-hv -> switches_no[0]-2
- U21 pad 12: adc-DRDY -> DRDY
- U5 pad 14: pi_cap_digital-power-hv -> hv
- U6 pad 2: comp_capacitor-power-hv -> switches_no[0]-2
- U8 pad 11: io[18]-line -> TXD
- U8 pad 19: touch[11]-MOSI -> host_spi-MOSI
- U8 pad 20: touch[12]-SCLK -> host_spi-SCLK
- U8 pad 21: touch[13]-MISO -> host_spi-MISO
- U8 pad 23: io[21]-23 -> io[21]-line
- U8 pad 31: 31 -> io[38]-line
- U8 pad 32: 32 -> io[39]-line
Routing:
- net 0: track 86.3 -> 131.5 mm, vias 16 -> 28
- net ch0-16: track 0.00 -> 38.8 mm, vias 0 -> 4
- net 161: track 38.8 -> 0.00 mm, vias 4 -> 0
- net power_3v3-hv: track 30.7 -> 0.00 mm, vias 8 -> 0
- net wifi_bypass_cap-power-hv: track 8.90 -> 0.00 mm
- net 80: track 0.00 -> 8.90 mm
- net hv: track 8.36 -> 0.00 mm
- net 248: track 0.00 -> 8.36 mm
- net host_in[2]-line: track 0.00 -> 8.20 mm
- net 235: track 8.20 -> 0.00 mm
- net OUTA: track 0.00 -> 3.21 mm
- net 112: track 3.21 -> 0.00 mm
- net ch0-7: track 0.00 -> 2.88 mm
- net 105: track 2.88 -> 0.00 mm
- added copper zone on F.Cu, net 6
- removed copper zone on F.Cu, net _inductor_2-6
